File: kicad/driver_64x64/driver.kicad_sch (KiCad schematic)
At the start: 0 parts

Commit message: logical seperation into host and multiple decode/drive/steering boards
Parts:
- added TP_ccs_channel_CCS_RET, TP_ccs_channel_ISENSE, TP_ccs_channel_VDRIVE, TP_decode_block_ADDR_NH (x3), TP_decode_block_ADDR_NL (x3), TP_decode_block_BANK_EN, TP_decode_block_DEC_EN, TP_decode_block_N_HS0_n, TP_decode_block_N_HS1_n, TP_decode_block_N_HS2_n, TP_decode_block_N_HS3_n, TP_decode_block_N_HS4_n, TP_decode_block_N_HS5_n, TP_decode_block_N_HS6_n, TP_decode_block_N_HS7_n, TP_decode_block_N_LS0_e, TP_decode_block_N_LS1_e, TP_decode_block_N_LS2_e, TP_decode_block_N_LS3_e, TP_decode_block_N_LS4_e, TP_decode_block_N_LS5_e, TP_decode_block_N_LS6_e, TP_decode_block_N_LS7_e, TP_dmos_hs_array_CCS_RE, TP_dmos_hs_array_IN0_n, TP_dmos_hs_array_IN1_n, TP_dmos_hs_array_IN2_n, TP_dmos_hs_array_IN3_n, TP_dmos_hs_array_IN4_n, TP_dmos_hs_array_IN5_n, TP_dmos_hs_array_IN6_n, TP_dmos_hs_array_IN7_n, TP_dmos_hs_array_OUT0, TP_dmos_hs_array_OUT1, TP_dmos_hs_array_OUT2, TP_dmos_hs_array_OUT3, TP_dmos_hs_array_OUT4, TP_dmos_hs_array_OUT5, TP_dmos_hs_array_OUT6, TP_dmos_hs_array_OUT7, TP_dmos_hs_array_VDRIVE, TP_dmos_ls_array_CCS_RE, TP_dmos_ls_array_IN0_en, TP_dmos_ls_array_IN1_en, TP_dmos_ls_array_IN2_en, TP_dmos_ls_array_IN3_en, TP_dmos_ls_array_IN4_en, TP_dmos_ls_array_IN5_en, TP_dmos_ls_array_IN6_en, TP_dmos_ls_array_IN7_en, TP_dmos_ls_array_OUT0, TP_dmos_ls_array_OUT1, TP_dmos_ls_array_OUT2, TP_dmos_ls_array_OUT3, TP_dmos_ls_array_OUT4, TP_dmos_ls_array_OUT5, TP_dmos_ls_array_OUT6, TP_dmos_ls_array_OUT7, TP_dmos_ls_array_VDRIVE, TP_magnetic_plane_SENSE, TP_magnetic_plane_XA0, TP_magnetic_plane_XA63, TP_magnetic_plane_XB0, TP_magnetic_plane_XB63, TP_magnetic_plane_YA0, TP_magnetic_plane_YA63, TP_magnetic_plane_YA65, TP_magnetic_plane_YA66, TP_magnetic_plane_YB0, TP_magnetic_plane_YB63, TP_magnetic_plane_YB65, TP_magnetic_plane_YB66, TP_sense_front_end_DOUT, TP_sense_front_end_INH_, TP_sense_front_end_PIO_, TP_sense_front_end_SENS, TP_sense_front_end_YA65, TP_sense_front_end_YB66, TP_steer_octal_X_g0_XA0, TP_steer_octal_X_g0_XA1, TP_steer_octal_X_g0_XA2, TP_steer_octal_X_g0_XA3, TP_steer_octal_X_g0_XA4, TP_steer_octal_X_g0_XA5, TP_steer_octal_X_g0_XA6, TP_steer_octal_X_g0_XA7, TP_steer_octal_X_g0_XB0, TP_steer_octal_X_g0_XB1, TP_steer_octal_X_g0_XB2, TP_steer_octal_X_g0_XB3, TP_steer_octal_X_g0_XB4, TP_steer_octal_X_g0_XB5, TP_steer_octal_X_g0_XB6, TP_steer_octal_X_g0_XB7, TP_steer_octal_X_g0_XHS (x2), TP_steer_octal_X_g0_XLS (x16), TP_steer_octal_X_g1_XA1 (x6), TP_steer_octal_X_g1_XA8, TP_steer_octal_X_g1_XA9, TP_steer_octal_X_g1_XB1 (x6), TP_steer_octal_X_g1_XB8, TP_steer_octal_X_g1_XB9, TP_steer_octal_X_g1_XHS (x2), TP_steer_octal_X_g1_XLS (x16), TP_steer_octal_X_g2_XA1 (x4), TP_steer_octal_X_g2_XA2 (x4), TP_steer_octal_X_g2_XB1 (x4), TP_steer_octal_X_g2_XB2 (x4), TP_steer_octal_X_g2_XHS (x2), TP_steer_octal_X_g2_XLS (x16), TP_steer_octal_X_g3_XA2 (x6), TP_steer_octal_X_g3_XA3 (x2), TP_steer_octal_X_g3_XB2 (x6), TP_steer_octal_X_g3_XB3 (x2), TP_steer_octal_X_g3_XHS (x2), TP_steer_octal_X_g3_XLS (x16), TP_steer_octal_X_g4_XA3 (x8), TP_steer_octal_X_g4_XB3 (x8), TP_steer_octal_X_g4_XHS (x2), TP_steer_octal_X_g4_XLS (x16), TP_steer_octal_X_g5_XA4 (x8), TP_steer_octal_X_g5_XB4 (x8), TP_steer_octal_X_g5_XHS (x2), TP_steer_octal_X_g5_XLS (x16), TP_steer_octal_X_g6_XA4 (x2), TP_steer_octal_X_g6_XA5 (x6), TP_steer_octal_X_g6_XB4 (x2), TP_steer_octal_X_g6_XB5 (x6), TP_steer_octal_X_g6_XHS (x2), TP_steer_octal_X_g6_XLS (x16), TP_steer_octal_X_g7_XA5 (x4), TP_steer_octal_X_g7_XA6 (x4), TP_steer_octal_X_g7_XB5 (x4), TP_steer_octal_X_g7_XB6 (x4), TP_steer_octal_X_g7_XHS (x2), TP_steer_octal_X_g7_XLS (x16), TP_steer_octal_Y_g0_YA0, TP_steer_octal_Y_g0_YA1, TP_steer_octal_Y_g0_YA2, TP_steer_octal_Y_g0_YA3, TP_steer_octal_Y_g0_YA4, TP_steer_octal_Y_g0_YA5, TP_steer_octal_Y_g0_YA6, TP_steer_octal_Y_g0_YA7, TP_steer_octal_Y_g0_YB0, TP_steer_octal_Y_g0_YB1, TP_steer_octal_Y_g0_YB2, TP_steer_octal_Y_g0_YB3, TP_steer_octal_Y_g0_YB4, TP_steer_octal_Y_g0_YB5, TP_steer_octal_Y_g0_YB6, TP_steer_octal_Y_g0_YB7, TP_steer_octal_Y_g0_YHS (x2), TP_steer_octal_Y_g0_YLS (x16), TP_steer_octal_Y_g1_YA1 (x6), TP_steer_octal_Y_g1_YA8, TP_steer_octal_Y_g1_YA9, TP_steer_octal_Y_g1_YB1 (x6), TP_steer_octal_Y_g1_YB8, TP_steer_octal_Y_g1_YB9, TP_steer_octal_Y_g1_YHS (x2), TP_steer_octal_Y_g1_YLS (x16), TP_steer_octal_Y_g2_YA1 (x4), TP_steer_octal_Y_g2_YA2 (x4), TP_steer_octal_Y_g2_YB1 (x4), TP_steer_octal_Y_g2_YB2 (x4), TP_steer_octal_Y_g2_YHS (x2), TP_steer_octal_Y_g2_YLS (x16), TP_steer_octal_Y_g3_YA2 (x6), TP_steer_octal_Y_g3_YA3 (x2), TP_steer_octal_Y_g3_YB2 (x6), TP_steer_octal_Y_g3_YB3 (x2), TP_steer_octal_Y_g3_YHS (x2), TP_steer_octal_Y_g3_YLS (x16), TP_steer_octal_Y_g4_YA3 (x8), TP_steer_octal_Y_g4_YB3 (x8), TP_steer_octal_Y_g4_YHS (x2), TP_steer_octal_Y_g4_YLS (x16), TP_steer_octal_Y_g5_YA4 (x8), TP_steer_octal_Y_g5_YB4 (x8), TP_steer_octal_Y_g5_YHS (x2), TP_steer_octal_Y_g5_YLS (x16), TP_steer_octal_Y_g6_YA4 (x2), TP_steer_octal_Y_g6_YA5 (x6), TP_steer_octal_Y_g6_YB4 (x2), TP_steer_octal_Y_g6_YB5 (x6), TP_steer_octal_Y_g6_YHS (x2), TP_steer_octal_Y_g6_YLS (x16), TP_steer_octal_Y_g7_YA5 (x4), TP_steer_octal_Y_g7_YA6 (x4), TP_steer_octal_Y_g7_YB5 (x4), TP_steer_octal_Y_g7_YB6 (x4), TP_steer_octal_Y_g7_YHS (x2), TP_steer_octal_Y_g7_YLS (x16): Stub, symbol CMR:Stub
Connections:
- net ccs_channel/CCS_RET: now also TP_ccs_channel_CCS_RET.1
- net ccs_channel/ISENSE: now also TP_ccs_channel_ISENSE.1
- net ccs_channel/VDRIVE: now also TP_ccs_channel_VDRIVE.1
- net decode_block/ADDR_NH0: now also TP_decode_block_ADDR_NH.1
- net decode_block/ADDR_NH1: now also TP_decode_block_ADDR_NH.1
- net decode_block/ADDR_NH2: now also TP_decode_block_ADDR_NH.1
- net decode_block/ADDR_NL0: now also TP_decode_block_ADDR_NL.1
- net decode_block/ADDR_NL1: now also TP_decode_block_ADDR_NL.1
- net decode_block/ADDR_NL2: now also TP_decode_block_ADDR_NL.1
- net decode_block/BANK_EN: now also TP_decode_block_BANK_EN.1
- net decode_block/DEC_EN: now also TP_decode_block_DEC_EN.1
- net decode_block/N_HS0_n: now also TP_decode_block_N_HS0_n.1
- net decode_block/N_HS1_n: now also TP_decode_block_N_HS1_n.1
- net decode_block/N_HS2_n: now also TP_decode_block_N_HS2_n.1
- net decode_block/N_HS3_n: now also TP_decode_block_N_HS3_n.1
- net decode_block/N_HS4_n: now also TP_decode_block_N_HS4_n.1
- net decode_block/N_HS5_n: now also TP_decode_block_N_HS5_n.1
- net decode_block/N_HS6_n: now also TP_decode_block_N_HS6_n.1
- net decode_block/N_HS7_n: now also TP_decode_block_N_HS7_n.1
- net decode_block/N_LS0_en: now also TP_decode_block_N_LS0_e.1
- net decode_block/N_LS1_en: now also TP_decode_block_N_LS1_e.1
- net decode_block/N_LS2_en: now also TP_decode_block_N_LS2_e.1
- net decode_block/N_LS3_en: now also TP_decode_block_N_LS3_e.1
- net decode_block/N_LS4_en: now also TP_decode_block_N_LS4_e.1
- net decode_block/N_LS5_en: now also TP_decode_block_N_LS5_e.1
- net decode_block/N_LS6_en: now also TP_decode_block_N_LS6_e.1
- net decode_block/N_LS7_en: now also TP_decode_block_N_LS7_e.1
- net dmos_hs_array/CCS_RET: now also TP_dmos_hs_array_CCS_RE.1
- net dmos_hs_array/IN0_n: now also TP_dmos_hs_array_IN0_n.1
- net dmos_hs_array/IN1_n: now also TP_dmos_hs_array_IN1_n.1
- net dmos_hs_array/IN2_n: now also TP_dmos_hs_array_IN2_n.1
- net dmos_hs_array/IN3_n: now also TP_dmos_hs_array_IN3_n.1
- net dmos_hs_array/IN4_n: now also TP_dmos_hs_array_IN4_n.1
- net dmos_hs_array/IN5_n: now also TP_dmos_hs_array_IN5_n.1
- net dmos_hs_array/IN6_n: now also TP_dmos_hs_array_IN6_n.1
- net dmos_hs_array/IN7_n: now also TP_dmos_hs_array_IN7_n.1
- net dmos_hs_array/OUT0: now also TP_dmos_hs_array_OUT0.1
- net dmos_hs_array/OUT1: now also TP_dmos_hs_array_OUT1.1
- net dmos_hs_array/OUT2: now also TP_dmos_hs_array_OUT2.1
- net dmos_hs_array/OUT3: now also TP_dmos_hs_array_OUT3.1
- net dmos_hs_array/OUT4: now also TP_dmos_hs_array_OUT4.1
- net dmos_hs_array/OUT5: now also TP_dmos_hs_array_OUT5.1
- net dmos_hs_array/OUT6: now also TP_dmos_hs_array_OUT6.1
- net dmos_hs_array/OUT7: now also TP_dmos_hs_array_OUT7.1
- net dmos_hs_array/VDRIVE: now also TP_dmos_hs_array_VDRIVE.1
- net dmos_ls_array/CCS_RET: now also TP_dmos_ls_array_CCS_RE.1
- net dmos_ls_array/IN0_en: now also TP_dmos_ls_array_IN0_en.1
- net dmos_ls_array/IN1_en: now also TP_dmos_ls_array_IN1_en.1
- net dmos_ls_array/IN2_en: now also TP_dmos_ls_array_IN2_en.1
- net dmos_ls_array/IN3_en: now also TP_dmos_ls_array_IN3_en.1
- net dmos_ls_array/IN4_en: now also TP_dmos_ls_array_IN4_en.1
- net dmos_ls_array/IN5_en: now also TP_dmos_ls_array_IN5_en.1
- net dmos_ls_array/IN6_en: now also TP_dmos_ls_array_IN6_en.1
- net dmos_ls_array/IN7_en: now also TP_dmos_ls_array_IN7_en.1
- net dmos_ls_array/OUT0: now also TP_dmos_ls_array_OUT0.1
- net dmos_ls_array/OUT1: now also TP_dmos_ls_array_OUT1.1
- net dmos_ls_array/OUT2: now also TP_dmos_ls_array_OUT2.1
- net dmos_ls_array/OUT3: now also TP_dmos_ls_array_OUT3.1
- net dmos_ls_array/OUT4: now also TP_dmos_ls_array_OUT4.1
- net dmos_ls_array/OUT5: now also TP_dmos_ls_array_OUT5.1
- net dmos_ls_array/OUT6: now also TP_dmos_ls_array_OUT6.1
- net dmos_ls_array/OUT7: now also TP_dmos_ls_array_OUT7.1
- net dmos_ls_array/VDRIVE: now also TP_dmos_ls_array_VDRIVE.1
- net magnetic_plane/SENSE_FOLD: now also TP_magnetic_plane_SENSE.1
- net magnetic_plane/XA0: now also TP_magnetic_plane_XA0.1
- net magnetic_plane/XA63: now also TP_magnetic_plane_XA63.1
- net magnetic_plane/XB0: now also TP_magnetic_plane_XB0.1
- net magnetic_plane/XB63: now also TP_magnetic_plane_XB63.1
- net magnetic_plane/YA0: now also TP_magnetic_plane_YA0.1
- net magnetic_plane/YA63: now also TP_magnetic_plane_YA63.1
- net magnetic_plane/YA65: now also TP_magnetic_plane_YA65.1
- net magnetic_plane/YA66: now also TP_magnetic_plane_YA66.1
- net magnetic_plane/YB0: now also TP_magnetic_plane_YB0.1
- net magnetic_plane/YB63: now also TP_magnetic_plane_YB63.1
- net magnetic_plane/YB65: now also TP_magnetic_plane_YB65.1
- net magnetic_plane/YB66: now also TP_magnetic_plane_YB66.1
- net sense_front_end/DOUT: now also TP_sense_front_end_DOUT.1
- net sense_front_end/INH_POL_SEL: now also TP_sense_front_end_INH_.1
- net sense_front_end/PIO_STROBE: now also TP_sense_front_end_PIO_.1
- net sense_front_end/SENSE_STROBE: now also TP_sense_front_end_SENS.1
- net sense_front_end/YA65: now also TP_sense_front_end_YA65.1
- net sense_front_end/YB66: now also TP_sense_front_end_YB66.1
- net steer_octal_X_g0/XA0: now also TP_steer_octal_X_g0_XA0.1
- net steer_octal_X_g0/XA1: now also TP_steer_octal_X_g0_XA1.1
- net steer_octal_X_g0/XA2: now also TP_steer_octal_X_g0_XA2.1
- net steer_octal_X_g0/XA3: now also TP_steer_octal_X_g0_XA3.1
- net steer_octal_X_g0/XA4: now also TP_steer_octal_X_g0_XA4.1
- net steer_octal_X_g0/XA5: now also TP_steer_octal_X_g0_XA5.1
- net steer_octal_X_g0/XA6: now also TP_steer_octal_X_g0_XA6.1
- net steer_octal_X_g0/XA7: now also TP_steer_octal_X_g0_XA7.1
- net steer_octal_X_g0/XB0: now also TP_steer_octal_X_g0_XB0.1
- net steer_octal_X_g0/XB1: now also TP_steer_octal_X_g0_XB1.1
- net steer_octal_X_g0/XB2: now also TP_steer_octal_X_g0_XB2.1
- net steer_octal_X_g0/XB3: now also TP_steer_octal_X_g0_XB3.1
- net steer_octal_X_g0/XB4: now also TP_steer_octal_X_g0_XB4.1
- net steer_octal_X_g0/XB5: now also TP_steer_octal_X_g0_XB5.1
- net steer_octal_X_g0/XB6: now also TP_steer_octal_X_g0_XB6.1
- net steer_octal_X_g0/XB7: now also TP_steer_octal_X_g0_XB7.1
- net steer_octal_X_g0/XHS0: now also TP_steer_octal_X_g0_XHS.1
- net steer_octal_X_g0/XHS0R: now also TP_steer_octal_X_g0_XHS.1
- net steer_octal_X_g0/XLS0: now also TP_steer_octal_X_g0_XLS.1
- net steer_octal_X_g0/XLS0R: now also TP_steer_octal_X_g0_XLS.1
- net steer_octal_X_g0/XLS1: now also TP_steer_octal_X_g0_XLS.1
- net steer_octal_X_g0/XLS1R: now also TP_steer_octal_X_g0_XLS.1
- net steer_octal_X_g0/XLS2: now also TP_steer_octal_X_g0_XLS.1
- net steer_octal_X_g0/XLS2R: now also TP_steer_octal_X_g0_XLS.1
- net steer_octal_X_g0/XLS3: now also TP_steer_octal_X_g0_XLS.1
- net steer_octal_X_g0/XLS3R: now also TP_steer_octal_X_g0_XLS.1
- net steer_octal_X_g0/XLS4: now also TP_steer_octal_X_g0_XLS.1
- net steer_octal_X_g0/XLS4R: now also TP_steer_octal_X_g0_XLS.1
- net steer_octal_X_g0/XLS5: now also TP_steer_octal_X_g0_XLS.1
- net steer_octal_X_g0/XLS5R: now also TP_steer_octal_X_g0_XLS.1
- net steer_octal_X_g0/XLS6: now also TP_steer_octal_X_g0_XLS.1
- net steer_octal_X_g0/XLS6R: now also TP_steer_octal_X_g0_XLS.1
- net steer_octal_X_g0/XLS7: now also TP_steer_octal_X_g0_XLS.1
- net steer_octal_X_g0/XLS7R: now also TP_steer_octal_X_g0_XLS.1
- net steer_octal_X_g1/XA10: now also TP_steer_octal_X_g1_XA1.1
- net steer_octal_X_g1/XA11: now also TP_steer_octal_X_g1_XA1.1
- net steer_octal_X_g1/XA12: now also TP_steer_octal_X_g1_XA1.1
- net steer_octal_X_g1/XA13: now also TP_steer_octal_X_g1_XA1.1
- net steer_octal_X_g1/XA14: now also TP_steer_octal_X_g1_XA1.1
- net steer_octal_X_g1/XA15: now also TP_steer_octal_X_g1_XA1.1
- net steer_octal_X_g1/XA8: now also TP_steer_octal_X_g1_XA8.1
- net steer_octal_X_g1/XA9: now also TP_steer_octal_X_g1_XA9.1
- net steer_octal_X_g1/XB10: now also TP_steer_octal_X_g1_XB1.1
- net steer_octal_X_g1/XB11: now also TP_steer_octal_X_g1_XB1.1
- net steer_octal_X_g1/XB12: now also TP_steer_octal_X_g1_XB1.1
- net steer_octal_X_g1/XB13: now also TP_steer_octal_X_g1_XB1.1
- net steer_octal_X_g1/XB14: now also TP_steer_octal_X_g1_XB1.1
- net steer_octal_X_g1/XB15: now also TP_steer_octal_X_g1_XB1.1
- net steer_octal_X_g1/XB8: now also TP_steer_octal_X_g1_XB8.1
- net steer_octal_X_g1/XB9: now also TP_steer_octal_X_g1_XB9.1
- net steer_octal_X_g1/XHS1: now also TP_steer_octal_X_g1_XHS.1
- net steer_octal_X_g1/XHS1R: now also TP_steer_octal_X_g1_XHS.1
- net steer_octal_X_g1/XLS0: now also TP_steer_octal_X_g1_XLS.1
- net steer_octal_X_g1/XLS0R: now also TP_steer_octal_X_g1_XLS.1
- net steer_octal_X_g1/XLS1: now also TP_steer_octal_X_g1_XLS.1
- net steer_octal_X_g1/XLS1R: now also TP_steer_octal_X_g1_XLS.1
- net steer_octal_X_g1/XLS2: now also TP_steer_octal_X_g1_XLS.1
- net steer_octal_X_g1/XLS2R: now also TP_steer_octal_X_g1_XLS.1
- net steer_octal_X_g1/XLS3: now also TP_steer_octal_X_g1_XLS.1
- net steer_octal_X_g1/XLS3R: now also TP_steer_octal_X_g1_XLS.1
- net steer_octal_X_g1/XLS4: now also TP_steer_octal_X_g1_XLS.1
- net steer_octal_X_g1/XLS4R: now also TP_steer_octal_X_g1_XLS.1
- net steer_octal_X_g1/XLS5: now also TP_steer_octal_X_g1_XLS.1
- net steer_octal_X_g1/XLS5R: now also TP_steer_octal_X_g1_XLS.1
- net steer_octal_X_g1/XLS6: now also TP_steer_octal_X_g1_XLS.1
- net steer_octal_X_g1/XLS6R: now also TP_steer_octal_X_g1_XLS.1
- net steer_octal_X_g1/XLS7: now also TP_steer_octal_X_g1_XLS.1
- net steer_octal_X_g1/XLS7R: now also TP_steer_octal_X_g1_XLS.1
- net steer_octal_X_g2/XA16: now also TP_steer_octal_X_g2_XA1.1
- net steer_octal_X_g2/XA17: now also TP_steer_octal_X_g2_XA1.1
- net steer_octal_X_g2/XA18: now also TP_steer_octal_X_g2_XA1.1
- net steer_octal_X_g2/XA19: now also TP_steer_octal_X_g2_XA1.1
- net steer_octal_X_g2/XA20: now also TP_steer_octal_X_g2_XA2.1
- net steer_octal_X_g2/XA21: now also TP_steer_octal_X_g2_XA2.1
- net steer_octal_X_g2/XA22: now also TP_steer_octal_X_g2_XA2.1
- net steer_octal_X_g2/XA23: now also TP_steer_octal_X_g2_XA2.1
- net steer_octal_X_g2/XB16: now also TP_steer_octal_X_g2_XB1.1
- net steer_octal_X_g2/XB17: now also TP_steer_octal_X_g2_XB1.1
- net steer_octal_X_g2/XB18: now also TP_steer_octal_X_g2_XB1.1
- net steer_octal_X_g2/XB19: now also TP_steer_octal_X_g2_XB1.1
- net steer_octal_X_g2/XB20: now also TP_steer_octal_X_g2_XB2.1
- net steer_octal_X_g2/XB21: now also TP_steer_octal_X_g2_XB2.1
- net steer_octal_X_g2/XB22: now also TP_steer_octal_X_g2_XB2.1
- net steer_octal_X_g2/XB23: now also TP_steer_octal_X_g2_XB2.1
- net steer_octal_X_g2/XHS2: now also TP_steer_octal_X_g2_XHS.1
- net steer_octal_X_g2/XHS2R: now also TP_steer_octal_X_g2_XHS.1
- net steer_octal_X_g2/XLS0: now also TP_steer_octal_X_g2_XLS.1
- net steer_octal_X_g2/XLS0R: now also TP_steer_octal_X_g2_XLS.1
- net steer_octal_X_g2/XLS1: now also TP_steer_octal_X_g2_XLS.1
- net steer_octal_X_g2/XLS1R: now also TP_steer_octal_X_g2_XLS.1
- net steer_octal_X_g2/XLS2: now also TP_steer_octal_X_g2_XLS.1
- net steer_octal_X_g2/XLS2R: now also TP_steer_octal_X_g2_XLS.1
- net steer_octal_X_g2/XLS3: now also TP_steer_octal_X_g2_XLS.1
- net steer_octal_X_g2/XLS3R: now also TP_steer_octal_X_g2_XLS.1
- net steer_octal_X_g2/XLS4: now also TP_steer_octal_X_g2_XLS.1
- net steer_octal_X_g2/XLS4R: now also TP_steer_octal_X_g2_XLS.1
- net steer_octal_X_g2/XLS5: now also TP_steer_octal_X_g2_XLS.1
- net steer_octal_X_g2/XLS5R: now also TP_steer_octal_X_g2_XLS.1
- net steer_octal_X_g2/XLS6: now also TP_steer_octal_X_g2_XLS.1
- net steer_octal_X_g2/XLS6R: now also TP_steer_octal_X_g2_XLS.1
- net steer_octal_X_g2/XLS7: now also TP_steer_octal_X_g2_XLS.1
- net steer_octal_X_g2/XLS7R: now also TP_steer_octal_X_g2_XLS.1
- net steer_octal_X_g3/XA24: now also TP_steer_octal_X_g3_XA2.1
- net steer_octal_X_g3/XA25: now also TP_steer_octal_X_g3_XA2.1
- net steer_octal_X_g3/XA26: now also TP_steer_octal_X_g3_XA2.1
- net steer_octal_X_g3/XA27: now also TP_steer_octal_X_g3_XA2.1
- net steer_octal_X_g3/XA28: now also TP_steer_octal_X_g3_XA2.1
- net steer_octal_X_g3/XA29: now also TP_steer_octal_X_g3_XA2.1
- net steer_octal_X_g3/XA30: now also TP_steer_octal_X_g3_XA3.1
- net steer_octal_X_g3/XA31: now also TP_steer_octal_X_g3_XA3.1
- net steer_octal_X_g3/XB24: now also TP_steer_octal_X_g3_XB2.1
- net steer_octal_X_g3/XB25: now also TP_steer_octal_X_g3_XB2.1
- net steer_octal_X_g3/XB26: now also TP_steer_octal_X_g3_XB2.1
- net steer_octal_X_g3/XB27: now also TP_steer_octal_X_g3_XB2.1
- net steer_octal_X_g3/XB28: now also TP_steer_octal_X_g3_XB2.1
- net steer_octal_X_g3/XB29: now also TP_steer_octal_X_g3_XB2.1
- net steer_octal_X_g3/XB30: now also TP_steer_octal_X_g3_XB3.1
- net steer_octal_X_g3/XB31: now also TP_steer_octal_X_g3_XB3.1
- net steer_octal_X_g3/XHS3: now also TP_steer_octal_X_g3_XHS.1
- net steer_octal_X_g3/XHS3R: now also TP_steer_octal_X_g3_XHS.1
- net steer_octal_X_g3/XLS0: now also TP_steer_octal_X_g3_XLS.1
- net steer_octal_X_g3/XLS0R: now also TP_steer_octal_X_g3_XLS.1
- net steer_octal_X_g3/XLS1: now also TP_steer_octal_X_g3_XLS.1
- net steer_octal_X_g3/XLS1R: now also TP_steer_octal_X_g3_XLS.1
- net steer_octal_X_g3/XLS2: now also TP_steer_octal_X_g3_XLS.1
- net steer_octal_X_g3/XLS2R: now also TP_steer_octal_X_g3_XLS.1
- net steer_octal_X_g3/XLS3: now also TP_steer_octal_X_g3_XLS.1
- net steer_octal_X_g3/XLS3R: now also TP_steer_octal_X_g3_XLS.1
- net steer_octal_X_g3/XLS4: now also TP_steer_octal_X_g3_XLS.1
- net steer_octal_X_g3/XLS4R: now also TP_steer_octal_X_g3_XLS.1
- net steer_octal_X_g3/XLS5: now also TP_steer_octal_X_g3_XLS.1
- net steer_octal_X_g3/XLS5R: now also TP_steer_octal_X_g3_XLS.1
- net steer_octal_X_g3/XLS6: now also TP_steer_octal_X_g3_XLS.1
- net steer_octal_X_g3/XLS6R: now also TP_steer_octal_X_g3_XLS.1
- net steer_octal_X_g3/XLS7: now also TP_steer_octal_X_g3_XLS.1
- net steer_octal_X_g3/XLS7R: now also TP_steer_octal_X_g3_XLS.1
- net steer_octal_X_g4/XA32: now also TP_steer_octal_X_g4_XA3.1
- net steer_octal_X_g4/XA33: now also TP_steer_octal_X_g4_XA3.1
- net steer_octal_X_g4/XA34: now also TP_steer_octal_X_g4_XA3.1
- net steer_octal_X_g4/XA35: now also TP_steer_octal_X_g4_XA3.1
- net steer_octal_X_g4/XA36: now also TP_steer_octal_X_g4_XA3.1
- net steer_octal_X_g4/XA37: now also TP_steer_octal_X_g4_XA3.1
- net steer_octal_X_g4/XA38: now also TP_steer_octal_X_g4_XA3.1
- net steer_octal_X_g4/XA39: now also TP_steer_octal_X_g4_XA3.1
- net steer_octal_X_g4/XB32: now also TP_steer_octal_X_g4_XB3.1
- net steer_octal_X_g4/XB33: now also TP_steer_octal_X_g4_XB3.1
- net steer_octal_X_g4/XB34: now also TP_steer_octal_X_g4_XB3.1
- net steer_octal_X_g4/XB35: now also TP_steer_octal_X_g4_XB3.1
- net steer_octal_X_g4/XB36: now also TP_steer_octal_X_g4_XB3.1
- net steer_octal_X_g4/XB37: now also TP_steer_octal_X_g4_XB3.1
- net steer_octal_X_g4/XB38: now also TP_steer_octal_X_g4_XB3.1
- net steer_octal_X_g4/XB39: now also TP_steer_octal_X_g4_XB3.1
- net steer_octal_X_g4/XHS4: now also TP_steer_octal_X_g4_XHS.1
- net steer_octal_X_g4/XHS4R: now also TP_steer_octal_X_g4_XHS.1
- net steer_octal_X_g4/XLS0: now also TP_steer_octal_X_g4_XLS.1
- net steer_octal_X_g4/XLS0R: now also TP_steer_octal_X_g4_XLS.1
- net steer_octal_X_g4/XLS1: now also TP_steer_octal_X_g4_XLS.1
- net steer_octal_X_g4/XLS1R: now also TP_steer_octal_X_g4_XLS.1
- net steer_octal_X_g4/XLS2: now also TP_steer_octal_X_g4_XLS.1
- net steer_octal_X_g4/XLS2R: now also TP_steer_octal_X_g4_XLS.1
- net steer_octal_X_g4/XLS3: now also TP_steer_octal_X_g4_XLS.1
- net steer_octal_X_g4/XLS3R: now also TP_steer_octal_X_g4_XLS.1
- net steer_octal_X_g4/XLS4: now also TP_steer_octal_X_g4_XLS.1
- net steer_octal_X_g4/XLS4R: now also TP_steer_octal_X_g4_XLS.1
- net steer_octal_X_g4/XLS5: now also TP_steer_octal_X_g4_XLS.1
- net steer_octal_X_g4/XLS5R: now also TP_steer_octal_X_g4_XLS.1
- net steer_octal_X_g4/XLS6: now also TP_steer_octal_X_g4_XLS.1
- net steer_octal_X_g4/XLS6R: now also TP_steer_octal_X_g4_XLS.1
- net steer_octal_X_g4/XLS7: now also TP_steer_octal_X_g4_XLS.1
- net steer_octal_X_g4/XLS7R: now also TP_steer_octal_X_g4_XLS.1
- net steer_octal_X_g5/XA40: now also TP_steer_octal_X_g5_XA4.1
- net steer_octal_X_g5/XA41: now also TP_steer_octal_X_g5_XA4.1
- net steer_octal_X_g5/XA42: now also TP_steer_octal_X_g5_XA4.1
- net steer_octal_X_g5/XA43: now also TP_steer_octal_X_g5_XA4.1
- net steer_octal_X_g5/XA44: now also TP_steer_octal_X_g5_XA4.1
- net steer_octal_X_g5/XA45: now also TP_steer_octal_X_g5_XA4.1
- net steer_octal_X_g5/XA46: now also TP_steer_octal_X_g5_XA4.1
- net steer_octal_X_g5/XA47: now also TP_steer_octal_X_g5_XA4.1
- net steer_octal_X_g5/XB40: now also TP_steer_octal_X_g5_XB4.1
- net steer_octal_X_g5/XB41: now also TP_steer_octal_X_g5_XB4.1
- net steer_octal_X_g5/XB42: now also TP_steer_octal_X_g5_XB4.1
- net steer_octal_X_g5/XB43: now also TP_steer_octal_X_g5_XB4.1
- net steer_octal_X_g5/XB44: now also TP_steer_octal_X_g5_XB4.1
- net steer_octal_X_g5/XB45: now also TP_steer_octal_X_g5_XB4.1
- net steer_octal_X_g5/XB46: now also TP_steer_octal_X_g5_XB4.1
- net steer_octal_X_g5/XB47: now also TP_steer_octal_X_g5_XB4.1
- net steer_octal_X_g5/XHS5: now also TP_steer_octal_X_g5_XHS.1
- net steer_octal_X_g5/XHS5R: now also TP_steer_octal_X_g5_XHS.1
- net steer_octal_X_g5/XLS0: now also TP_steer_octal_X_g5_XLS.1
- net steer_octal_X_g5/XLS0R: now also TP_steer_octal_X_g5_XLS.1
- net steer_octal_X_g5/XLS1: now also TP_steer_octal_X_g5_XLS.1
- net steer_octal_X_g5/XLS1R: now also TP_steer_octal_X_g5_XLS.1
- net steer_octal_X_g5/XLS2: now also TP_steer_octal_X_g5_XLS.1
- net steer_octal_X_g5/XLS2R: now also TP_steer_octal_X_g5_XLS.1
- net steer_octal_X_g5/XLS3: now also TP_steer_octal_X_g5_XLS.1
- net steer_octal_X_g5/XLS3R: now also TP_steer_octal_X_g5_XLS.1
- net steer_octal_X_g5/XLS4: now also TP_steer_octal_X_g5_XLS.1
- net steer_octal_X_g5/XLS4R: now also TP_steer_octal_X_g5_XLS.1
- net steer_octal_X_g5/XLS5: now also TP_steer_octal_X_g5_XLS.1
- net steer_octal_X_g5/XLS5R: now also TP_steer_octal_X_g5_XLS.1
- net steer_octal_X_g5/XLS6: now also TP_steer_octal_X_g5_XLS.1
- net steer_octal_X_g5/XLS6R: now also TP_steer_octal_X_g5_XLS.1
- net steer_octal_X_g5/XLS7: now also TP_steer_octal_X_g5_XLS.1
- net steer_octal_X_g5/XLS7R: now also TP_steer_octal_X_g5_XLS.1
- net steer_octal_X_g6/XA48: now also TP_steer_octal_X_g6_XA4.1
- net steer_octal_X_g6/XA49: now also TP_steer_octal_X_g6_XA4.1
- net steer_octal_X_g6/XA50: now also TP_steer_octal_X_g6_XA5.1
- net steer_octal_X_g6/XA51: now also TP_steer_octal_X_g6_XA5.1
- net steer_octal_X_g6/XA52: now also TP_steer_octal_X_g6_XA5.1
- net steer_octal_X_g6/XA53: now also TP_steer_octal_X_g6_XA5.1
- net steer_octal_X_g6/XA54: now also TP_steer_octal_X_g6_XA5.1
- net steer_octal_X_g6/XA55: now also TP_steer_octal_X_g6_XA5.1
- net steer_octal_X_g6/XB48: now also TP_steer_octal_X_g6_XB4.1
- net steer_octal_X_g6/XB49: now also TP_steer_octal_X_g6_XB4.1
- net steer_octal_X_g6/XB50: now also TP_steer_octal_X_g6_XB5.1
- net steer_octal_X_g6/XB51: now also TP_steer_octal_X_g6_XB5.1
- net steer_octal_X_g6/XB52: now also TP_steer_octal_X_g6_XB5.1
- net steer_octal_X_g6/XB53: now also TP_steer_octal_X_g6_XB5.1
- net steer_octal_X_g6/XB54: now also TP_steer_octal_X_g6_XB5.1
- net steer_octal_X_g6/XB55: now also TP_steer_octal_X_g6_XB5.1
- net steer_octal_X_g6/XHS6: now also TP_steer_octal_X_g6_XHS.1
- net steer_octal_X_g6/XHS6R: now also TP_steer_octal_X_g6_XHS.1
- net steer_octal_X_g6/XLS0: now also TP_steer_octal_X_g6_XLS.1
- net steer_octal_X_g6/XLS0R: now also TP_steer_octal_X_g6_XLS.1
- net steer_octal_X_g6/XLS1: now also TP_steer_octal_X_g6_XLS.1
- net steer_octal_X_g6/XLS1R: now also TP_steer_octal_X_g6_XLS.1
- net steer_octal_X_g6/XLS2: now also TP_steer_octal_X_g6_XLS.1
- net steer_octal_X_g6/XLS2R: now also TP_steer_octal_X_g6_XLS.1
- net steer_octal_X_g6/XLS3: now also TP_steer_octal_X_g6_XLS.1
- net steer_octal_X_g6/XLS3R: now also TP_steer_octal_X_g6_XLS.1
- net steer_octal_X_g6/XLS4: now also TP_steer_octal_X_g6_XLS.1
- net steer_octal_X_g6/XLS4R: now also TP_steer_octal_X_g6_XLS.1
- net steer_octal_X_g6/XLS5: now also TP_steer_octal_X_g6_XLS.1
- net steer_octal_X_g6/XLS5R: now also TP_steer_octal_X_g6_XLS.1
- net steer_octal_X_g6/XLS6: now also TP_steer_octal_X_g6_XLS.1
- net steer_octal_X_g6/XLS6R: now also TP_steer_octal_X_g6_XLS.1
- net steer_octal_X_g6/XLS7: now also TP_steer_octal_X_g6_XLS.1
- net steer_octal_X_g6/XLS7R: now also TP_steer_octal_X_g6_XLS.1
- net steer_octal_X_g7/XA56: now also TP_steer_octal_X_g7_XA5.1
- net steer_octal_X_g7/XA57: now also TP_steer_octal_X_g7_XA5.1
- net steer_octal_X_g7/XA58: now also TP_steer_octal_X_g7_XA5.1
- net steer_octal_X_g7/XA59: now also TP_steer_octal_X_g7_XA5.1
- net steer_octal_X_g7/XA60: now also TP_steer_octal_X_g7_XA6.1
- net steer_octal_X_g7/XA61: now also TP_steer_octal_X_g7_XA6.1
- net steer_octal_X_g7/XA62: now also TP_steer_octal_X_g7_XA6.1
- net steer_octal_X_g7/XA63: now also TP_steer_octal_X_g7_XA6.1
- net steer_octal_X_g7/XB56: now also TP_steer_octal_X_g7_XB5.1
- net steer_octal_X_g7/XB57: now also TP_steer_octal_X_g7_XB5.1
- net steer_octal_X_g7/XB58: now also TP_steer_octal_X_g7_XB5.1
- net steer_octal_X_g7/XB59: now also TP_steer_octal_X_g7_XB5.1
- net steer_octal_X_g7/XB60: now also TP_steer_octal_X_g7_XB6.1
- net steer_octal_X_g7/XB61: now also TP_steer_octal_X_g7_XB6.1
- net steer_octal_X_g7/XB62: now also TP_steer_octal_X_g7_XB6.1
- net steer_octal_X_g7/XB63: now also TP_steer_octal_X_g7_XB6.1
- net steer_octal_X_g7/XHS7: now also TP_steer_octal_X_g7_XHS.1
- net steer_octal_X_g7/XHS7R: now also TP_steer_octal_X_g7_XHS.1
- net steer_octal_X_g7/XLS0: now also TP_steer_octal_X_g7_XLS.1
- net steer_octal_X_g7/XLS0R: now also TP_steer_octal_X_g7_XLS.1
- net steer_octal_X_g7/XLS1: now also TP_steer_octal_X_g7_XLS.1
- net steer_octal_X_g7/XLS1R: now also TP_steer_octal_X_g7_XLS.1
- net steer_octal_X_g7/XLS2: now also TP_steer_octal_X_g7_XLS.1
- net steer_octal_X_g7/XLS2R: now also TP_steer_octal_X_g7_XLS.1
- net steer_octal_X_g7/XLS3: now also TP_steer_octal_X_g7_XLS.1
- net steer_octal_X_g7/XLS3R: now also TP_steer_octal_X_g7_XLS.1
- net steer_octal_X_g7/XLS4: now also TP_steer_octal_X_g7_XLS.1
- net steer_octal_X_g7/XLS4R: now also TP_steer_octal_X_g7_XLS.1
- net steer_octal_X_g7/XLS5: now also TP_steer_octal_X_g7_XLS.1
- net steer_octal_X_g7/XLS5R: now also TP_steer_octal_X_g7_XLS.1
- net steer_octal_X_g7/XLS6: now also TP_steer_octal_X_g7_XLS.1
- net steer_octal_X_g7/XLS6R: now also TP_steer_octal_X_g7_XLS.1
- net steer_octal_X_g7/XLS7: now also TP_steer_octal_X_g7_XLS.1
- net steer_octal_X_g7/XLS7R: now also TP_steer_octal_X_g7_XLS.1
- net steer_octal_Y_g0/YA0: now also TP_steer_octal_Y_g0_YA0.1
- net steer_octal_Y_g0/YA1: now also TP_steer_octal_Y_g0_YA1.1
- net steer_octal_Y_g0/YA2: now also TP_steer_octal_Y_g0_YA2.1
- net steer_octal_Y_g0/YA3: now also TP_steer_octal_Y_g0_YA3.1
- net steer_octal_Y_g0/YA4: now also TP_steer_octal_Y_g0_YA4.1
- net steer_octal_Y_g0/YA5: now also TP_steer_octal_Y_g0_YA5.1
- net steer_octal_Y_g0/YA6: now also TP_steer_octal_Y_g0_YA6.1
- net steer_octal_Y_g0/YA7: now also TP_steer_octal_Y_g0_YA7.1
- net steer_octal_Y_g0/YB0: now also TP_steer_octal_Y_g0_YB0.1
- net steer_octal_Y_g0/YB1: now also TP_steer_octal_Y_g0_YB1.1
- net steer_octal_Y_g0/YB2: now also TP_steer_octal_Y_g0_YB2.1
- net steer_octal_Y_g0/YB3: now also TP_steer_octal_Y_g0_YB3.1
- net steer_octal_Y_g0/YB4: now also TP_steer_octal_Y_g0_YB4.1
- net steer_octal_Y_g0/YB5: now also TP_steer_octal_Y_g0_YB5.1
- net steer_octal_Y_g0/YB6: now also TP_steer_octal_Y_g0_YB6.1
- net steer_octal_Y_g0/YB7: now also TP_steer_octal_Y_g0_YB7.1
- net steer_octal_Y_g0/YHS0: now also TP_steer_octal_Y_g0_YHS.1
- net steer_octal_Y_g0/YHS0R: now also TP_steer_octal_Y_g0_YHS.1
- net steer_octal_Y_g0/YLS0: now also TP_steer_octal_Y_g0_YLS.1
- net steer_octal_Y_g0/YLS0R: now also TP_steer_octal_Y_g0_YLS.1
- net steer_octal_Y_g0/YLS1: now also TP_steer_octal_Y_g0_YLS.1
- net steer_octal_Y_g0/YLS1R: now also TP_steer_octal_Y_g0_YLS.1
- net steer_octal_Y_g0/YLS2: now also TP_steer_octal_Y_g0_YLS.1
- net steer_octal_Y_g0/YLS2R: now also TP_steer_octal_Y_g0_YLS.1
- net steer_octal_Y_g0/YLS3: now also TP_steer_octal_Y_g0_YLS.1
- net steer_octal_Y_g0/YLS3R: now also TP_steer_octal_Y_g0_YLS.1
- net steer_octal_Y_g0/YLS4: now also TP_steer_octal_Y_g0_YLS.1
- net steer_octal_Y_g0/YLS4R: now also TP_steer_octal_Y_g0_YLS.1
- net steer_octal_Y_g0/YLS5: now also TP_steer_octal_Y_g0_YLS.1
- net steer_octal_Y_g0/YLS5R: now also TP_steer_octal_Y_g0_YLS.1
- net steer_octal_Y_g0/YLS6: now also TP_steer_octal_Y_g0_YLS.1
- net steer_octal_Y_g0/YLS6R: now also TP_steer_octal_Y_g0_YLS.1
- net steer_octal_Y_g0/YLS7: now also TP_steer_octal_Y_g0_YLS.1
- net steer_octal_Y_g0/YLS7R: now also TP_steer_octal_Y_g0_YLS.1
- net steer_octal_Y_g1/YA10: now also TP_steer_octal_Y_g1_YA1.1
- net steer_octal_Y_g1/YA11: now also TP_steer_octal_Y_g1_YA1.1
- net steer_octal_Y_g1/YA12: now also TP_steer_octal_Y_g1_YA1.1
- net steer_octal_Y_g1/YA13: now also TP_steer_octal_Y_g1_YA1.1
- net steer_octal_Y_g1/YA14: now also TP_steer_octal_Y_g1_YA1.1
- net steer_octal_Y_g1/YA15: now also TP_steer_octal_Y_g1_YA1.1
- net steer_octal_Y_g1/YA8: now also TP_steer_octal_Y_g1_YA8.1
- net steer_octal_Y_g1/YA9: now also TP_steer_octal_Y_g1_YA9.1
- net steer_octal_Y_g1/YB10: now also TP_steer_octal_Y_g1_YB1.1
- net steer_octal_Y_g1/YB11: now also TP_steer_octal_Y_g1_YB1.1
- net steer_octal_Y_g1/YB12: now also TP_steer_octal_Y_g1_YB1.1
- net steer_octal_Y_g1/YB13: now also TP_steer_octal_Y_g1_YB1.1
- net steer_octal_Y_g1/YB14: now also TP_steer_octal_Y_g1_YB1.1
- net steer_octal_Y_g1/YB15: now also TP_steer_octal_Y_g1_YB1.1
- net steer_octal_Y_g1/YB8: now also TP_steer_octal_Y_g1_YB8.1
- net steer_octal_Y_g1/YB9: now also TP_steer_octal_Y_g1_YB9.1
- net steer_octal_Y_g1/YHS1: now also TP_steer_octal_Y_g1_YHS.1
- net steer_octal_Y_g1/YHS1R: now also TP_steer_octal_Y_g1_YHS.1
- net steer_octal_Y_g1/YLS0: now also TP_steer_octal_Y_g1_YLS.1
- net steer_octal_Y_g1/YLS0R: now also TP_steer_octal_Y_g1_YLS.1
- net steer_octal_Y_g1/YLS1: now also TP_steer_octal_Y_g1_YLS.1
- net steer_octal_Y_g1/YLS1R: now also TP_steer_octal_Y_g1_YLS.1
- net steer_octal_Y_g1/YLS2: now also TP_steer_octal_Y_g1_YLS.1
- net steer_octal_Y_g1/YLS2R: now also TP_steer_octal_Y_g1_YLS.1
- net steer_octal_Y_g1/YLS3: now also TP_steer_octal_Y_g1_YLS.1
- net steer_octal_Y_g1/YLS3R: now also TP_steer_octal_Y_g1_YLS.1
- net steer_octal_Y_g1/YLS4: now also TP_steer_octal_Y_g1_YLS.1
- net steer_octal_Y_g1/YLS4R: now also TP_steer_octal_Y_g1_YLS.1
- net steer_octal_Y_g1/YLS5: now also TP_steer_octal_Y_g1_YLS.1
- net steer_octal_Y_g1/YLS5R: now also TP_steer_octal_Y_g1_YLS.1
- net steer_octal_Y_g1/YLS6: now also TP_steer_octal_Y_g1_YLS.1
- net steer_octal_Y_g1/YLS6R: now also TP_steer_octal_Y_g1_YLS.1
- net steer_octal_Y_g1/YLS7: now also TP_steer_octal_Y_g1_YLS.1
- net steer_octal_Y_g1/YLS7R: now also TP_steer_octal_Y_g1_YLS.1
- net steer_octal_Y_g2/YA16: now also TP_steer_octal_Y_g2_YA1.1
- net steer_octal_Y_g2/YA17: now also TP_steer_octal_Y_g2_YA1.1
- net steer_octal_Y_g2/YA18: now also TP_steer_octal_Y_g2_YA1.1
- net steer_octal_Y_g2/YA19: now also TP_steer_octal_Y_g2_YA1.1
- net steer_octal_Y_g2/YA20: now also TP_steer_octal_Y_g2_YA2.1
- net steer_octal_Y_g2/YA21: now also TP_steer_octal_Y_g2_YA2.1
- net steer_octal_Y_g2/YA22: now also TP_steer_octal_Y_g2_YA2.1
- net steer_octal_Y_g2/YA23: now also TP_steer_octal_Y_g2_YA2.1
- net steer_octal_Y_g2/YB16: now also TP_steer_octal_Y_g2_YB1.1
- net steer_octal_Y_g2/YB17: now also TP_steer_octal_Y_g2_YB1.1
- net steer_octal_Y_g2/YB18: now also TP_steer_octal_Y_g2_YB1.1
- net steer_octal_Y_g2/YB19: now also TP_steer_octal_Y_g2_YB1.1
- net steer_octal_Y_g2/YB20: now also TP_steer_octal_Y_g2_YB2.1
- net steer_octal_Y_g2/YB21: now also TP_steer_octal_Y_g2_YB2.1
- net steer_octal_Y_g2/YB22: now also TP_steer_octal_Y_g2_YB2.1
- net steer_octal_Y_g2/YB23: now also TP_steer_octal_Y_g2_YB2.1
- net steer_octal_Y_g2/YHS2: now also TP_steer_octal_Y_g2_YHS.1
- net steer_octal_Y_g2/YHS2R: now also TP_steer_octal_Y_g2_YHS.1
- net steer_octal_Y_g2/YLS0: now also TP_steer_octal_Y_g2_YLS.1
- net steer_octal_Y_g2/YLS0R: now also TP_steer_octal_Y_g2_YLS.1
- net steer_octal_Y_g2/YLS1: now also TP_steer_octal_Y_g2_YLS.1
- net steer_octal_Y_g2/YLS1R: now also TP_steer_octal_Y_g2_YLS.1
- net steer_octal_Y_g2/YLS2: now also TP_steer_octal_Y_g2_YLS.1
- net steer_octal_Y_g2/YLS2R: now also TP_steer_octal_Y_g2_YLS.1
- net steer_octal_Y_g2/YLS3: now also TP_steer_octal_Y_g2_YLS.1
- net steer_octal_Y_g2/YLS3R: now also TP_steer_octal_Y_g2_YLS.1
- net steer_octal_Y_g2/YLS4: now also TP_steer_octal_Y_g2_YLS.1
- net steer_octal_Y_g2/YLS4R: now also TP_steer_octal_Y_g2_YLS.1
- net steer_octal_Y_g2/YLS5: now also TP_steer_octal_Y_g2_YLS.1
- net steer_octal_Y_g2/YLS5R: now also TP_steer_octal_Y_g2_YLS.1
- net steer_octal_Y_g2/YLS6: now also TP_steer_octal_Y_g2_YLS.1
- net steer_octal_Y_g2/YLS6R: now also TP_steer_octal_Y_g2_YLS.1
- net steer_octal_Y_g2/YLS7: now also TP_steer_octal_Y_g2_YLS.1
- net steer_octal_Y_g2/YLS7R: now also TP_steer_octal_Y_g2_YLS.1
- net steer_octal_Y_g3/YA24: now also TP_steer_octal_Y_g3_YA2.1
- net steer_octal_Y_g3/YA25: now also TP_steer_octal_Y_g3_YA2.1
- net steer_octal_Y_g3/YA26: now also TP_steer_octal_Y_g3_YA2.1
- net steer_octal_Y_g3/YA27: now also TP_steer_octal_Y_g3_YA2.1
- net steer_octal_Y_g3/YA28: now also TP_steer_octal_Y_g3_YA2.1
- net steer_octal_Y_g3/YA29: now also TP_steer_octal_Y_g3_YA2.1
- net steer_octal_Y_g3/YA30: now also TP_steer_octal_Y_g3_YA3.1
- net steer_octal_Y_g3/YA31: now also TP_steer_octal_Y_g3_YA3.1
- net steer_octal_Y_g3/YB24: now also TP_steer_octal_Y_g3_YB2.1
- net steer_octal_Y_g3/YB25: now also TP_steer_octal_Y_g3_YB2.1
- net steer_octal_Y_g3/YB26: now also TP_steer_octal_Y_g3_YB2.1
- net steer_octal_Y_g3/YB27: now also TP_steer_octal_Y_g3_YB2.1
- net steer_octal_Y_g3/YB28: now also TP_steer_octal_Y_g3_YB2.1
- net steer_octal_Y_g3/YB29: now also TP_steer_octal_Y_g3_YB2.1
- net steer_octal_Y_g3/YB30: now also TP_steer_octal_Y_g3_YB3.1
- net steer_octal_Y_g3/YB31: now also TP_steer_octal_Y_g3_YB3.1
- net steer_octal_Y_g3/YHS3: now also TP_steer_octal_Y_g3_YHS.1
- net steer_octal_Y_g3/YHS3R: now also TP_steer_octal_Y_g3_YHS.1
- net steer_octal_Y_g3/YLS0: now also TP_steer_octal_Y_g3_YLS.1
- net steer_octal_Y_g3/YLS0R: now also TP_steer_octal_Y_g3_YLS.1
- net steer_octal_Y_g3/YLS1: now also TP_steer_octal_Y_g3_YLS.1
- net steer_octal_Y_g3/YLS1R: now also TP_steer_octal_Y_g3_YLS.1
- net steer_octal_Y_g3/YLS2: now also TP_steer_octal_Y_g3_YLS.1
- net steer_octal_Y_g3/YLS2R: now also TP_steer_octal_Y_g3_YLS.1
- net steer_octal_Y_g3/YLS3: now also TP_steer_octal_Y_g3_YLS.1
- net steer_octal_Y_g3/YLS3R: now also TP_steer_octal_Y_g3_YLS.1
- net steer_octal_Y_g3/YLS4: now also TP_steer_octal_Y_g3_YLS.1
- net steer_octal_Y_g3/YLS4R: now also TP_steer_octal_Y_g3_YLS.1
- net steer_octal_Y_g3/YLS5: now also TP_steer_octal_Y_g3_YLS.1
- net steer_octal_Y_g3/YLS5R: now also TP_steer_octal_Y_g3_YLS.1
- net steer_octal_Y_g3/YLS6: now also TP_steer_octal_Y_g3_YLS.1
- net steer_octal_Y_g3/YLS6R: now also TP_steer_octal_Y_g3_YLS.1
- net steer_octal_Y_g3/YLS7: now also TP_steer_octal_Y_g3_YLS.1
- net steer_octal_Y_g3/YLS7R: now also TP_steer_octal_Y_g3_YLS.1
- net steer_octal_Y_g4/YA32: now also TP_steer_octal_Y_g4_YA3.1
- net steer_octal_Y_g4/YA33: now also TP_steer_octal_Y_g4_YA3.1
- net steer_octal_Y_g4/YA34: now also TP_steer_octal_Y_g4_YA3.1
- net steer_octal_Y_g4/YA35: now also TP_steer_octal_Y_g4_YA3.1
- net steer_octal_Y_g4/YA36: now also TP_steer_octal_Y_g4_YA3.1
- net steer_octal_Y_g4/YA37: now also TP_steer_octal_Y_g4_YA3.1
- net steer_octal_Y_g4/YA38: now also TP_steer_octal_Y_g4_YA3.1
- net steer_octal_Y_g4/YA39: now also TP_steer_octal_Y_g4_YA3.1
- net steer_octal_Y_g4/YB32: now also TP_steer_octal_Y_g4_YB3.1
- net steer_octal_Y_g4/YB33: now also TP_steer_octal_Y_g4_YB3.1
- net steer_octal_Y_g4/YB34: now also TP_steer_octal_Y_g4_YB3.1
- net steer_octal_Y_g4/YB35: now also TP_steer_octal_Y_g4_YB3.1
- net steer_octal_Y_g4/YB36: now also TP_steer_octal_Y_g4_YB3.1
- net steer_octal_Y_g4/YB37: now also TP_steer_octal_Y_g4_YB3.1
- net steer_octal_Y_g4/YB38: now also TP_steer_octal_Y_g4_YB3.1
- net steer_octal_Y_g4/YB39: now also TP_steer_octal_Y_g4_YB3.1
- net steer_octal_Y_g4/YHS4: now also TP_steer_octal_Y_g4_YHS.1
- net steer_octal_Y_g4/YHS4R: now also TP_steer_octal_Y_g4_YHS.1
- net steer_octal_Y_g4/YLS0: now also TP_steer_octal_Y_g4_YLS.1
- net steer_octal_Y_g4/YLS0R: now also TP_steer_octal_Y_g4_YLS.1
- net steer_octal_Y_g4/YLS1: now also TP_steer_octal_Y_g4_YLS.1
- net steer_octal_Y_g4/YLS1R: now also TP_steer_octal_Y_g4_YLS.1
- net steer_octal_Y_g4/YLS2: now also TP_steer_octal_Y_g4_YLS.1
- net steer_octal_Y_g4/YLS2R: now also TP_steer_octal_Y_g4_YLS.1
- net steer_octal_Y_g4/YLS3: now also TP_steer_octal_Y_g4_YLS.1
- net steer_octal_Y_g4/YLS3R: now also TP_steer_octal_Y_g4_YLS.1
- net steer_octal_Y_g4/YLS4: now also TP_steer_octal_Y_g4_YLS.1
- net steer_octal_Y_g4/YLS4R: now also TP_steer_octal_Y_g4_YLS.1
- net steer_octal_Y_g4/YLS5: now also TP_steer_octal_Y_g4_YLS.1
- net steer_octal_Y_g4/YLS5R: now also TP_steer_octal_Y_g4_YLS.1
- net steer_octal_Y_g4/YLS6: now also TP_steer_octal_Y_g4_YLS.1
- net steer_octal_Y_g4/YLS6R: now also TP_steer_octal_Y_g4_YLS.1
- net steer_octal_Y_g4/YLS7: now also TP_steer_octal_Y_g4_YLS.1
- net steer_octal_Y_g4/YLS7R: now also TP_steer_octal_Y_g4_YLS.1
- net steer_octal_Y_g5/YA40: now also TP_steer_octal_Y_g5_YA4.1
- net steer_octal_Y_g5/YA41: now also TP_steer_octal_Y_g5_YA4.1
- net steer_octal_Y_g5/YA42: now also TP_steer_octal_Y_g5_YA4.1
- net steer_octal_Y_g5/YA43: now also TP_steer_octal_Y_g5_YA4.1
- net steer_octal_Y_g5/YA44: now also TP_steer_octal_Y_g5_YA4.1
- net steer_octal_Y_g5/YA45: now also TP_steer_octal_Y_g5_YA4.1
- net steer_octal_Y_g5/YA46: now also TP_steer_octal_Y_g5_YA4.1
- net steer_octal_Y_g5/YA47: now also TP_steer_octal_Y_g5_YA4.1
- net steer_octal_Y_g5/YB40: now also TP_steer_octal_Y_g5_YB4.1
- net steer_octal_Y_g5/YB41: now also TP_steer_octal_Y_g5_YB4.1
- net steer_octal_Y_g5/YB42: now also TP_steer_octal_Y_g5_YB4.1
- net steer_octal_Y_g5/YB43: now also TP_steer_octal_Y_g5_YB4.1
- net steer_octal_Y_g5/YB44: now also TP_steer_octal_Y_g5_YB4.1
- net steer_octal_Y_g5/YB45: now also TP_steer_octal_Y_g5_YB4.1
- net steer_octal_Y_g5/YB46: now also TP_steer_octal_Y_g5_YB4.1
- net steer_octal_Y_g5/YB47: now also TP_steer_octal_Y_g5_YB4.1
- net steer_octal_Y_g5/YHS5: now also TP_steer_octal_Y_g5_YHS.1
- net steer_octal_Y_g5/YHS5R: now also TP_steer_octal_Y_g5_YHS.1
- net steer_octal_Y_g5/YLS0: now also TP_steer_octal_Y_g5_YLS.1
- net steer_octal_Y_g5/YLS0R: now also TP_steer_octal_Y_g5_YLS.1
- net steer_octal_Y_g5/YLS1: now also TP_steer_octal_Y_g5_YLS.1
- net steer_octal_Y_g5/YLS1R: now also TP_steer_octal_Y_g5_YLS.1
- net steer_octal_Y_g5/YLS2: now also TP_steer_octal_Y_g5_YLS.1
- net steer_octal_Y_g5/YLS2R: now also TP_steer_octal_Y_g5_YLS.1
- net steer_octal_Y_g5/YLS3: now also TP_steer_octal_Y_g5_YLS.1
- net steer_octal_Y_g5/YLS3R: now also TP_steer_octal_Y_g5_YLS.1
- net steer_octal_Y_g5/YLS4: now also TP_steer_octal_Y_g5_YLS.1
- net steer_octal_Y_g5/YLS4R: now also TP_steer_octal_Y_g5_YLS.1
- net steer_octal_Y_g5/YLS5: now also TP_steer_octal_Y_g5_YLS.1
- net steer_octal_Y_g5/YLS5R: now also TP_steer_octal_Y_g5_YLS.1
- net steer_octal_Y_g5/YLS6: now also TP_steer_octal_Y_g5_YLS.1
- net steer_octal_Y_g5/YLS6R: now also TP_steer_octal_Y_g5_YLS.1
- net steer_octal_Y_g5/YLS7: now also TP_steer_octal_Y_g5_YLS.1
- net steer_octal_Y_g5/YLS7R: now also TP_steer_octal_Y_g5_YLS.1
- net steer_octal_Y_g6/YA48: now also TP_steer_octal_Y_g6_YA4.1
- net steer_octal_Y_g6/YA49: now also TP_steer_octal_Y_g6_YA4.1
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